Commit message: 同時に可視化をするように変更　値磁気センサのカルマンフィルタの実装　動作未確認

File: urdf/simple_drone.urdf (robot description, URDF)
Before this commit: robot simple_drone, 2 links, 1 joints
Links:
- removed link drone
- added link drone_kalman; visual box size=0.5 0.7 0.01
- added link drone_obse; visual box size=0.5 0.7 0.01
- added link drone_pred; visual box size=0.5 0.7 0.01
- added link obse_base
- added link pred_base
Joints:
- removed joint base_joint
- added joint base_joint_kalman: type floating, parent world, child drone_kalman
- added joint base_joint_obse: type floating, parent obse_base, child drone_obse
- added joint base_joint_pred: type floating, parent pred_base, child drone_pred
- added joint obse_joint: type fixed, parent world, child obse_base, origin xyz=-1.0 0.0 0.0 rpy=0.0 0.0 0.0
- added joint pred_joint: type fixed, parent world, child pred_base, origin xyz=1.0 0.0 0.0 rpy=0.0 0.0 0.0
